Commit message: Almost running

File: catkin_ws/src/custom_robot/urdf/custom_robot.xacro (robot description, xacro)
@@ -9,4 +9,6 @@
     </joint>
     <link name="base_plate">
+        <pose> 0 0 0.1 0 0 0 </pose>
+        <origin xyz="0.0 0.0 0.0" rpy="0.0 0.0 0.0"/>
         <inertial>
             <origin xyz="0.0 0.0 0.0" rpy="0.0 0.0 0.0"/>
@@ -15,11 +17,7 @@
         </inertial>
         <visual name="base_plate_visual">
-            <origin xyz="0.0 0.0 0.0" rpy="0.0 0.0 0.0"/>
             <geometry>
                 <mesh filename="package://custom_robot/meshes/BasePlate.dae"/>
             </geometry>
-            <material name="">
-                <color rgba="1.0 0.0 0.0 1.0"/>
-            </material>
         </visual>
         <collision>

Commit message: Still can't get visual to display in gazebo on custom_robot

File: catkin_ws/src/custom_robot/urdf/custom_robot.xacro (robot description, xacro)
@@ -28,3 +28,29 @@
         </collision>
     </link>
+    <link name="right_wheel">
+        <collision name="right_wheel_collision">
+            <origin xyz="0.0 0.0 0.0" rpy="0.0 1.5707 1.5707"/>
+            <geometry>
+                <cylinder radius="0.1" length="0.05"/>
+            </geometry>
+        </collision>
+        <visual name="right_wheel_visual">
+            <origin xyz="0.0 0.0 0.0" rpy="0.0 1.5707 1.5707"/>
+            <geometry>
+                <cylinder radius="0.1" length="0.05"/>
+            </geometry>
+        </visual>
+        <inertial>
+            <origin xyz="0.0 0.0 0.0" rpy="0.0 1.5707 1.5707"/>
+            <mass value="5"/>
+            <inertia ixx=".1" ixy="0" ixz="0" iyy="0.1" iyz="0.0" izz=".1"/>
+        </inertial>
+    </link>
+    <joint name="joint_name" type="continuous">
+        <origin xyz="0.0 0.0 0.0" rpy="0.0 0.0 0.0"/>
+        <parent link="base_plate"/>
+        <child link="right_wheel"/>
+        <axis xyz="0.0 0.0 0.0"/>
+        <limit lower="0.0" upper="0.0" effort="0.0" velocity="0.0"/>
+    </joint>
 </robot>

Commit message: half of model displayed in gazebo, fully in rviz

File: catkin_ws/src/custom_robot/urdf/custom_robot.xacro (robot description, xacro)
@@ -28,29 +28,303 @@
         </collision>
     </link>
-    <link name="right_wheel">
-        <collision name="right_wheel_collision">
-            <origin xyz="0.0 0.0 0.0" rpy="0.0 1.5707 1.5707"/>
+	<link name="right_wheel_hub">
+		<inertial>
+			<origin xyz="0.0 -0.25 0.0" rpy="0.0 0.0 0.0"/>
+			<mass value="0.0"/>
+			<inertia ixx="0.0" ixy="0.0" ixz="0.0" iyy="0.0" iyz="0.0" izz="0.0"/>
+		</inertial>
+		<visual name="right_wheel_hub_visual">
+			<origin xyz="0.0 -0.25 0.0" rpy="0.0 0.0 0.0"/>
+			<geometry>
+				<mesh filename="package://custom_robot/meshes/BearingMount.dae"/>
+			</geometry>
+		</visual>
+		<collision name="right_wheel_hub_collision">
+			<origin xyz="0.0 -0.25 0.0" rpy="0.0 0.0 0.0"/>
+			<geometry>
+				<cylinder radius="0.150" length="0.010"/>
+			</geometry>
+		</collision>
+	</link>
+	<joint name="right_wheel_hub_joint" type="fixed">
+		<origin xyz="0.0 0.0 0.0" rpy="0.0 0.0 0.0"/>
+		<parent link="base_plate"/>
+		<child link="right_wheel_hub"/>
+        <axis xyz="0.0 0.0 0.0"/>
+	</joint>
+	<link name="left_wheel_hub">
+		<inertial>
+			<origin xyz="0.0 0.25 0.0" rpy="0.0 0.0 0.0"/>
+			<mass value="0.0"/>
+			<inertia ixx="0.0" ixy="0.0" ixz="0.0" iyy="0.0" iyz="0.0" izz="0.0"/>
+		</inertial>
+		<visual name="left_wheel_hub_visual">
+			<origin xyz="0.0 0.25 0.0" rpy="0.0 0.0 0.0"/>
+			<geometry>
+				<mesh filename="package://custom_robot/meshes/BearingMount.dae"/>
+			</geometry>
+		</visual>
+		<collision name="left_wheel_hub_collision">
+			<origin xyz="0.0 0.25 0.0" rpy="0.0 0.0 0.0"/>
+			<geometry>
+				<cylinder radius="0.150" length="0.010"/>
+			</geometry>
+		</collision>
+	</link>
+	<joint name="left_wheel_hub_joint" type="fixed">
+		<origin xyz="0.0 0.0 0.0" rpy="0.0 0.0 0.0"/>
+		<parent link="base_plate"/>
+		<child link="left_wheel_hub"/>
+        <axis xyz="0.0 0.0 0.0"/>
+	</joint>
+	<link name="left_wheel_bearing">
+		<inertial>
+			<origin xyz="0.0  0.30 0.0" rpy="0.0 0.0 1.57"/>
+			<mass value="0.0"/>
+			<inertia ixx="0.0" ixy="0.0" ixz="0.0" iyy="0.0" iyz="0.0" izz="0.0"/>
+		</inertial>
+		<visual name="left_wheel_bearing_visual">
+			<origin xyz="0.0  0.30 0.0" rpy="0.0 0.0 1.57"/>
+			<geometry>
+				<mesh filename="package://custom_robot/meshes/WheelBearing.dae"/>
+			</geometry>
+		</visual>
+		<collision name="left_wheel_bearing_collision">
+			<origin xyz="0.0  0.30 0.0" rpy="0.0 0.0 1.57"/>
+			<geometry>
+				<cylinder radius="0.150" length="0.010"/>
+			</geometry>
+		</collision>
+	</link>
+	<joint name="left_wheel_bearing_joint" type="fixed">
+		<origin xyz="0.0 0.0 0.0" rpy="0.0 0.0 0.0"/>
+		<parent link="left_wheel_hub"/>
+		<child link="left_wheel_bearing"/>
+        <axis xyz="0.0 0.0 0.0"/>
+	</joint>
+	<link name="right_wheel_bearing">
+		<inertial>
+			<origin xyz="0.0 -0.30 0.0" rpy="0.0 0.0 1.57"/>
+			<mass value="0.0"/>
+			<inertia ixx="0.0" ixy="0.0" ixz="0.0" iyy="0.0" iyz="0.0" izz="0.0"/>
+		</inertial>
+		<visual name="left_wheel_bearing_visual">
+			<origin xyz="0.0 -0.30 0.0" rpy="0.0 0.0 1.57"/>
+			<geometry>
+				<mesh filename="package://custom_robot/meshes/WheelBearing.dae"/>
+			</geometry>
+		</visual>
+		<collision name="right_wheel_bearing_collision">
+			<origin xyz="0.0 -0.30 0.0" rpy="0.0 0.0 1.57"/>
+			<geometry>
+				<cylinder radius="0.150" length="0.010"/>
+			</geometry>
+		</collision>
+	</link>
+	<joint name="right_wheel_bearing_joint" type="fixed">
+		<origin xyz="0.0 0.0 0.0" rpy="0.0 0.0 0.0"/>
+		<parent link="right_wheel_hub"/>
+		<child link="right_wheel_bearing"/>
+        <axis xyz="0.0 0.0 0.0"/>
+	</joint>
+	<link name="right_wheel_shaft">
+		<inertial>
+			<origin xyz="0.0 -0.35 0.0" rpy="0.0 0.0 1.57"/>
+			<mass value="0.0"/>
+			<inertia ixx="0.0" ixy="0.0" ixz="0.0" iyy="0.0" iyz="0.0" izz="0.0"/>
+		</inertial>
+		<visual name="right_wheel_shaft_visual">
+			<origin xyz="0.0 -0.35 0.0" rpy="0.0 0.0 1.57"/>
+			<geometry>
+				<mesh filename="package://custom_robot/meshes/WheelShaft.dae"/>
+			</geometry>
+		</visual>
+		<collision name="right_wheel_shaft_collision">
+			<origin xyz="0.0 -0.35 0.0" rpy="0.0 0.0 1.57"/>
+			<geometry>
+				<cylinder radius="0.150" length="0.010"/>
+			</geometry>
+		</collision>
+	</link>
+	<joint name="right_wheel_shaft_joint" type="continuous">
+		<origin xyz="0.0 0.0 0.0" rpy="0.0 0.0 0.0"/>
+		<parent link="right_wheel_bearing"/>
+		<child link="right_wheel_shaft"/>
+        <axis xyz="0.0 1 0.0" rpy="0.0 0.0 0.0"/>
+        <limit effort="10000" velocity="1000"/>
+        <dynamics damping="1.0" friction="1.0"/>
+	</joint>
+	<link name="right_wheel">
+		<inertial>
+			<origin xyz="0.0 -0.5 0.0" rpy="0.0 0.0 0.0"/>
+			<mass value="0.0"/>
+			<inertia ixx="0.0" ixy="0.0" ixz="0.0" iyy="0.0" iyz="0.0" izz="0.0"/>
+		</inertial>
+		<visual name="right_wheel_visual">
+			<origin xyz="0.0 -0.5 0.0" rpy="0.0 0.0 0.0"/>
+			<geometry>
+				<mesh filename="package://custom_robot/meshes/Wheel.dae"/>
+			</geometry>
+		</visual>
+		<collision name="right_wheel_collision">
+			<origin xyz="0.0 -0.5 0.0" rpy="0.0 0.0 0.0"/>
+			<geometry>
+				<cylinder radius="150" length="10.0"/>
+			</geometry>
+		</collision>
+	</link>
+	<joint name="right_wheel_joint" type="fixed">
+		<origin xyz="0.0 0.0 0.0" rpy="0.0 0.0 0.0"/>
+		<parent link="right_wheel_shaft"/>
+		<child link="right_wheel"/>
+	</joint>
+	<link name="left_wheel_shaft">
+		<inertial>
+			<origin xyz="0.0  0.35 0.0" rpy="0.0 0.0 -1.57"/>
+			<mass value="0.0"/>
+			<inertia ixx="0.0" ixy="0.0" ixz="0.0" iyy="0.0" iyz="0.0" izz="0.0"/>
+		</inertial>
+		<visual name="left_wheel_shaft_visual">
+			<origin xyz="0.0  0.35 0.0" rpy="0.0 0.0 -1.57"/>
+			<geometry>
+				<mesh filename="package://custom_robot/meshes/WheelShaft.dae"/>
+			</geometry>
+		</visual>
+		<collision name="left_wheel_shaft_collision">
+			<origin xyz="0.0  0.35 0.0" rpy="0.0 0.0 -1.57"/>
+			<geometry>
+				<cylinder radius="0.150" length="0.010"/>
+			</geometry>
+		</collision>
+	</link>
+	<joint name="left_wheel_shaft_joint" type="continuous">
+		<origin xyz="0.0 0.0 0.0" rpy="0.0 0.0 0.0"/>
+		<parent link="left_wheel_bearing"/>
+		<child link="left_wheel_shaft"/>
+        <axis xyz="0.0 1 0.0" rpy="0.0 0.0 0.0"/>
+        <limit effort="10000" velocity="1000"/>
+        <dynamics damping="1.0" friction="1.0"/>
+	</joint>
+	<link name="left_wheel">
+		<inertial>
+			<origin xyz="0.0 0.5 0.0" rpy="0.0 0.0 0.0"/>
+			<mass value="0.0"/>
+			<inertia ixx="0.0" ixy="0.0" ixz="0.0" iyy="0.0" iyz="0.0" izz="0.0"/>
+		</inertial>
+		<visual name="left_wheel_visual">
+			<origin xyz="0.0 0.5 0.0" rpy="0.0 0.0 0.0"/>
+			<geometry>
+				<mesh filename="package://custom_robot/meshes/Wheel.dae"/>
+			</geometry>
+		</visual>
+		<collision name="left_wheel_collision">
+			<origin xyz="0.0 0.5 0.0" rpy="0.0 0.0 0.0"/>
+			<geometry>
+				<cylinder radius="150" length="10.0"/>
+			</geometry>
+		</collision>
+	</link>
+	<joint name="left_wheel_joint" type="fixed">
+		<origin xyz="0.0 0.0 0.0" rpy="0.0 0.0 0.0"/>
+		<parent link="left_wheel_shaft"/>
+		<child link="left_wheel"/>
+		<limit lower="0.0" upper="0.0" effort="0.0" velocity="0.0"/>
+	</joint>
+	<link name="left_timing_pulley">
+		<inertial>
+			<origin xyz="0.0  0.20 0.0" rpy="0.0 0.0 -1.57"/>
+			<mass value="0.0"/>
+			<inertia ixx="0.0" ixy="0.0" ixz="0.0" iyy="0.0" iyz="0.0" izz="0.0"/>
+		</inertial>
+		<visual name="left_timing_pulley_visual">
+			<origin xyz="0.0  0.20 0.0" rpy="0.0 0.0 -1.57"/>
+			<geometry>
+				<mesh filename="package://custom_robot/meshes/TimingPulley.dae"/>
+			</geometry>
+		</visual>
+		<collision name="left_timing_pulley_collision">
+			<origin xyz="0.0  0.20 0.0" rpy="0.0 0.0 -1.57"/>
+			<geometry>
+				<cylinder radius="0.150" length="0.010"/>
+			</geometry>
+		</collision>
+	</link>
+	<joint name="left_timing_pulley_joint" type="fixed">
+		<origin xyz="0.0 0.0 0.0" rpy="0.0 0.0 0.0"/>
+		<parent link="left_wheel_shaft"/>
+		<child link="left_timing_pulley"/>
+	</joint>
+	<link name="right_timing_pulley">
+		<inertial>
+			<origin xyz="0.0  0.20 0.0" rpy="0.0 0.0 -1.57"/>
+			<mass value="0.0"/>
+			<inertia ixx="0.0" ixy="0.0" ixz="0.0" iyy="0.0" iyz="0.0" izz="0.0"/>
+		</inertial>
+		<visual name="right_timing_pulley_visual">
+			<origin xyz="0.0  0.20 0.0" rpy="0.0 0.0 -1.57"/>
+			<geometry>
+				<mesh filename="package://custom_robot/meshes/TimingPulley.dae"/>
+			</geometry>
+		</visual>
+		<collision name="right_timing_pulley_collision">
+			<origin xyz="0.0  0.20 0.0" rpy="0.0 0.0 -1.57"/>
+			<geometry>
+				<cylinder radius="0.150" length="0.010"/>
+			</geometry>
+		</collision>
+	</link>
+	<joint name="right_timing_pulley_joint" type="fixed">
+		<origin xyz="0.0 0.0 0.0" rpy="0.0 0.0 0.0"/>
+		<parent link="right_wheel_shaft"/>
+		<child link="right_timing_pulley"/>
+	</joint>
+	<link name="test_object">
+		<inertial>
+			<origin xyz="0.0  0.20 0.0" rpy="0.0 0.0 -1.57"/>
+			<mass value="0.0"/>
+			<inertia ixx="0.0" ixy="0.0" ixz="0.0" iyy="0.0" iyz="0.0" izz="0.0"/>
+		</inertial>
+		<visual name="test_object_visual">
+			<origin xyz="0.0  0.20 0.0" rpy="0.0 0.0 -1.57"/>
+			<geometry>
+				<box size="0.001 0.001 0.001"/>
+			</geometry>
+		</visual>
+		<collision name="test_object_collision">
+			<origin xyz="0.0  0.20 0.0" rpy="0.0 0.0 -1.57"/>
+			<geometry>
+				<box size="0.001 0.001 0.001"/>
+			</geometry>
+		</collision>
+	</link>
+	<joint name="test_object_joint" type="fixed">
+		<origin xyz="0.0 0.0 0.0" rpy="0.0 0.0 0.0"/>
+		<parent link="base_plate"/>
+		<child link="test_object"/>
+	</joint>
+	<link name="hokuyo">
+        <origin xyz="0.0 0.0 0.0" rpy="0.0 0.0 0.0"/>
+        <inertial>
+            <mass value="1e-5"/>
+            <inertia ixx="1e-6" ixy="0.0" ixz="0.0" iyy="1e-6" iyz="0.0" izz="1e-6"/>
+        </inertial>
+        <visual name="hokuyo_visual">
+            <!-- <origin xyz="0.0 0.0 0.0" rpy="0.0 0.0 0.0"/> -->
             <geometry>
-                <cylinder radius="0.1" length="0.05"/>
+                <mesh filename="package://custom_robot/meshes/hokuyo.dae"/>
+            </geometry>
+        </visual>
+        <collision name="hokuyo_collision">
+            <origin xyz="0.0 0.0 0.0" rpy="0.0 0.0 0.0"/>
+            <geometry>
+                <box size=".1 .1 .1"/>
             </geometry>
         </collision>
-        <visual name="right_wheel_visual">
-            <origin xyz="0.0 0.0 0.0" rpy="0.0 1.5707 1.5707"/>
-            <geometry>
-                <cylinder radius="0.1" length="0.05"/>
-            </geometry>
-        </visual>
-        <inertial>
-            <origin xyz="0.0 0.0 0.0" rpy="0.0 1.5707 1.5707"/>
-            <mass value="5"/>
-            <inertia ixx=".1" ixy="0" ixz="0" iyy="0.1" iyz="0.0" izz=".1"/>
-        </inertial>
     </link>
-    <joint name="joint_name" type="continuous">
-        <origin xyz="0.0 0.0 0.0" rpy="0.0 0.0 0.0"/>
+    <joint name="hokuyo_joint" type="fixed">
+        <origin xyz="0.15 0.0 .1" rpy="0.0 0.0 0.0"/>
         <parent link="base_plate"/>
-        <child link="right_wheel"/>
-        <axis xyz="0.0 0.0 0.0"/>
-        <limit lower="0.0" upper="0.0" effort="0.0" velocity="0.0"/>
+        <child link="hokuyo"/>
+        <axis xyz="0.0 1 0.0"/>
     </joint>
 </robot>

Commit message: removed textures from DAE, added STL

File: catkin_ws/src/custom_robot/urdf/custom_robot.xacro (robot description, xacro)
@@ -51,5 +51,5 @@
 		<parent link="base_plate"/>
 		<child link="right_wheel_hub"/>
-        <axis xyz="0.0 0.0 0.0"/>
+        <axis xyz="0.0 1.0 0.0"/>
 	</joint>
 	<link name="left_wheel_hub">
@@ -178,4 +178,5 @@
 		<parent link="right_wheel_shaft"/>
 		<child link="right_wheel"/>
+        <axis xyz="0.0 1 0.0"/>
 	</joint>
 	<link name="left_wheel_shaft">
@@ -229,5 +230,5 @@
 		<parent link="left_wheel_shaft"/>
 		<child link="left_wheel"/>
-		<limit lower="0.0" upper="0.0" effort="0.0" velocity="0.0"/>
+        <axis xyz="0.0 1 0.0"/>
 	</joint>
 	<link name="left_timing_pulley">
@@ -328,3 +329,59 @@
         <axis xyz="0.0 1 0.0"/>
     </joint>
+    <link name="camera">
+        <inertial>
+            <origin xyz="0.0 0.0 0.0" rpy="0.0 0.0 0.0"/>
+            <mass value=".1"/>
+            <box_inertia m="0.1" x="0.05" y="0.05" z="0.05"/>
+            <inertia ixx="0.0" ixy="0.0" ixz="0.0" iyy="0.0" iyz="0.0" izz="0.0"/>
+        </inertial>
+        <visual name="">
+            <origin xyz="0.0 0.0 0.0" rpy="0.0 0.0 0.0"/>
+            <geometry>
+                <box size="0.05 0.05 0.05"/>
+            </geometry>
+        </visual>
+        <collision>
+            <origin xyz="0.0 0.0 0.0" rpy="0.0 0.0 0.0"/>
+            <geometry>
+                <box size="0.05 0.05 0.05"/>
+            </geometry>
+        </collision>
+    </link>
+    <joint name="camera_joint" type="fixed">
+        <origin xyz="0.0 0.0 0.0" rpy="0.0 0.0 0.0"/>
+        <parent link="base_plate"/>
+        <child link="camera"/>
+        <axis xyz="0.0 1.0 0.0"/>
+    </joint>
+    <link name="stupid_bot">
+        <inertial>
+            <origin xyz="5.0 5.0 0.0" rpy="0.0 0.0 0.0"/>
+            <mass value="0.0"/>
+            <inertia ixx="0.0" ixy="0.0" ixz="0.0" iyy="0.0" iyz="0.0" izz="0.0"/>
+        </inertial>
+        <visual name="stupid_bot_visual">
+            <origin xyz="5.0 5.0 0.0" rpy="0.0 0.0 0.0"/>
+            <geometry>
+                <mesh filename="package://custom_robot/meshes/Robot.dae"/>
+            </geometry>
+            <material name="">
+                <color rgba="1.0 0.0 0.0 1.0"/>
+                <texture filename=""/>
+            </material>
+        </visual>
+        <collision name="stupid_bot_collision">
+            <origin xyz="5.0 5.0 0.0" rpy="0.0 0.0 0.0"/>
+            <geometry>
+                <box size="1.0 1.0 1.0"/>
+            </geometry>
+        </collision>
+    </link>
+    <joint name="stupid_bot_joint" type="fixed">
+        <origin xyz="0.0 0.0 0.0" rpy="0.0 0.0 0.0"/>
+        <parent link="base_plate"/>
+        <child link="stupid_bot"/>
+        <axis xyz="0.0 0.0 0.0"/>
+        <limit lower="0.0" upper="0.0" effort="0.0" velocity="0.0"/>
+    </joint>
 </robot>

File: catkin_ws/src/my_robot/urdf/my_robot.xacro (robot description, xacro)
@@ -109,4 +109,30 @@
         </collision>
     </link>
+    <link name="camera">
+        <inertial>
+            <origin xyz="0.0 0.0 0.0" rpy="0.0 0.0 0.0"/>
+            <mass value="0.1"/>
+            <box_inertia m="0.1" x="0.05" y="0.05" z="0.05"/>
+            <inertia ixx="1e-6" ixy="0.0" ixz="0.0" iyy="1e-6" iyz="0.0" izz="1e-6"/>
+        </inertial>
+        <visual name="camera_visual">
+            <origin xyz="0.0 0.0 0.0" rpy="0.0 0.0 0.0"/>
+            <geometry>
+                <box size="0.05 0.05 0.05"/>
+            </geometry>
+        </visual>
+        <collision>
+            <origin xyz="0.0 0.0 0.0" rpy="0.0 0.0 0.0"/>
+            <geometry>
+                <box size="0.05 0.05 0.05"/>
+            </geometry>
+        </collision>
+    </link>
+    <joint name="camera_joint" type="fixed">
+        <origin xyz="0.2 0.0 0.0" rpy="0.0 0.0 0.0"/>
+        <parent link="chassis"/>
+        <child link="camera"/>
+        <axis xyz="0.0 1.0 0.0"/>
+    </joint>
     <joint name="hokuyo_joint" type="fixed">
         <origin xyz="0.15 0.0 .1" rpy="0.0 0.0 0.0"/>
