Commit message: Decent progress made on finished xacro

File: catkin_ws/src/wheel_bot_description/urdf/frame.xacro (robot description, xacro)
@@ -1,10 +1,137 @@
-	<?<?xml version="1.0"?>
-	<robot name="wheel_bot">
-		<link name="base_link">
-			<visual>
+<?xml version="1.0"?>
+	<robot name="wheel_bot" xmlns:xacro="http://www.ros.org/wiki/xacro">
+		<link name="base_link"></link>
+		<link name="base_plate_link">
+			<inertial>
+				<origin xyz="0.0 0.0 0.0" rpy="0.0 0.0 0.0"/>
+				<mass value="0.1"/>
+				<inertia ixx="0.1" ixy="0.0" ixz="0.0" iyy="0.1" iyz="0.0" izz="0.1"/>
+			</inertial>
+			<visual name="">
+				<origin xyz="0.0 0.0 0.0" rpy="0.0 0.0 0.0"/>
 				<geometry>
-					<cylinder radius="0.6" length="0.2"/>
+					<mesh filename="package://wheel_bot_description/meshes/BasePlate.dae" />
 				</geometry>
 			</visual>
+			<collision name="base_plate_collision">
+				<origin xyz="0.0 0.0 0.0" rpy="0.0 0.0 0.0"/>
+				<geometry>
+					<box size="0.1 0.1 0.1"/>
+				</geometry>
+			</collision>
 		</link>
-	</robot>
+		<joint name="base_to_base_plate" type="fixed">
+			<origin xyz="0.0 0.0 0.0" rpy="1.57075 0.0 0.0"/>
+			<parent link="base_link"/>
+			<child link="base_plate_link"/>
+			<axis xyz="0.0 0.0 0.0"/>
+			<limit lower="0.0" upper="0.0" effort="0.0" velocity="0.0"/>
+		</joint>
+		<link name="l_wheel_hub">
+			<inertial>
+				<origin xyz="0.0 0.0 0.0" rpy="0.0 0.0 0.0"/>
+				<mass value="0.1"/>
+				<inertia ixx="0.1" ixy="0.0" ixz="0.0" iyy="0.1" iyz="0.0" izz="0.1"/>
+			</inertial>
+			<visual name="l_wheel_hub_visual">
+				<origin xyz="0.0 0.0 0.0" rpy="0.0 0.0 0.0"/>
+					<geometry>
+						<mesh filename="package://wheel_bot_description/meshes/WheelHub.dae" />
+					</geometry>
+			</visual>
+			<collision name="l_wheel_hub_collision">
+				<origin xyz="0.0 0.0 0.0" rpy="0.0 0.0 0.0"/>
+				<geometry>
+					<box size="0.1 0.1 0.1"/>
+				</geometry>
+			</collision>
+		</link>
+		<joint name="l_hub_to_base_plate" type="fixed">
+			<origin xyz="0.1 0.025 0.150" rpy="0.0 3.14 0.0"/>
+			<parent link="base_plate_link"/>
+			<child link="l_wheel_hub"/>
+			<axis xyz="0.0 0.0 0.0"/>
+			<limit lower="0.0" upper="0.0" effort="0.0" velocity="0.0"/>
+		</joint>
+		<link name="l_wheel_bearing">
+			<inertial>
+				<origin xyz="0.0 0.0 0.0" rpy="0.0 0.0 0.0"/>
+				<mass value="0.1"/>
+				<inertia ixx="0.1" ixy="0.0" ixz="0.0" iyy="0.1" iyz="0.0" izz="0.1"/>
+			</inertial>
+			<visual name="l_wheel_bearing_visual">
+				<origin xyz="0.0 0.0 0.0" rpy="0.0 0.0 0.0"/>
+					<geometry>
+						<mesh filename="package://wheel_bot_description/meshes/WheelBearing.dae" />
+					</geometry>
+			</visual>
+			<collision name="l_wheel_bearing_collision">
+				<origin xyz="0.0 0.0 0.0" rpy="0.0 0.0 0.0"/>
+				<geometry>
+					<box size="0.1 0.1 0.1"/>
+				</geometry>
+			</collision>
+		</link>
+		<joint name="l_bearing_to_hub" type="fixed">
+			<origin xyz="0.025 0.080 0.010" rpy="0.0 1.57075 0.0"/>
+			<parent link="l_wheel_hub"/>
+			<child link="l_wheel_bearing"/>
+			<axis xyz="0.0 0.0 0.0"/>
+			<limit lower="0.0" upper="0.0" effort="0.0" velocity="0.0"/>
+		</joint>
+		<link name="l_wheel_shaft">
+			<inertial>
+				<origin xyz="0.0 0.0 0.0" rpy="0.0 0.0 0.0"/>
+				<mass value="0.1"/>
+				<inertia ixx="0.1" ixy="0.0" ixz="0.0" iyy="0.1" iyz="0.0" izz="0.1"/>
+			</inertial>
+			<visual name="l_wheel_shaft_visual">
+				<origin xyz="0.0 0.0 0.0" rpy="0.0 0.0 0.0"/>
+					<geometry>
+						<mesh filename="package://wheel_bot_description/meshes/WheelShaft.dae" />
+					</geometry>
+			</visual>
+			<collision name="l_wheel_shaft_collision">
+				<origin xyz="0.0 0.0 0.0" rpy="0.0 0.0 0.0"/>
+				<geometry>
+					<box size="0.1 0.1 0.1"/>
+				</geometry>
+			</collision>
+		</link>
+		<joint name="l_shaft_to_bearing" type="continuous">
+			<origin xyz="0.0 0.0 0.0" rpy="0.0 0.0 0.0"/>
+			<parent link="l_wheel_bearing"/>
+			<child link="l_wheel_shaft"/>
+			<axis xyz="1.0 0.0 0.0"/>
+			<limit lower="0.0" upper="0.0" effort="0.0" velocity="0.0"/>
+		</joint>
+		<link name="l_wheel">
+			<inertial>
+				<origin xyz="0.0 0.0 0.0" rpy="0.0 0.0 0.0"/>
+				<mass value="0.1"/>
+				<inertia ixx="0.1" ixy="0.0" ixz="0.0" iyy="0.1" iyz="0.0" izz="0.1"/>
+			</inertial>
+			<visual name="l_wheel_visual">
+				<origin xyz="0.0 0.0 0.0" rpy="0.0 0.0 0.0"/>
+					<geometry>
+						<mesh filename="package://wheel_bot_description/meshes/Wheel.dae" />
+					</geometry>
+			</visual>
+			<collision name="l_wheel_collision">
+				<origin xyz="0.0 0.0 0.0" rpy="0.0 0.0 0.0"/>
+				<geometry>
+					<mesh filename="package://wheel_bot_description/meshes/Wheel.dae" />
+				</geometry>
+				<!-- <geometry>
+					<box size="0.1 0.1 0.1"/>
+				</geometry> -->
+			</collision>
+		</link>
+		<joint name="l_wheel_to_shaft" type="fixed">
+			<origin xyz="0.0 0.0 0.0" rpy="0.0 1.57075 0.0"/>
+			<parent link="l_wheel_shaft"/>
+			<child link="l_wheel"/>
+			<axis xyz="0.0 0.0 0.0"/>
+			<limit lower="0.0" upper="0.0" effort="0.0" velocity="0.0"/>
+		</joint>
+</robot>

Commit message: right wheel side completed with approximate collision

File: catkin_ws/src/wheel_bot_description/urdf/frame.xacro (robot description, xacro)
@@ -5,8 +5,8 @@
 			<inertial>
 				<origin xyz="0.0 0.0 0.0" rpy="0.0 0.0 0.0"/>
-				<mass value="0.1"/>
-				<inertia ixx="0.1" ixy="0.0" ixz="0.0" iyy="0.1" iyz="0.0" izz="0.1"/>
+				<mass value="5.403"/>
+				<inertia ixx="0.000013" ixy="0.0" ixz="0.0" iyy="0.000026" iyz="0.0" izz="0.000013"/>
 			</inertial>
-			<visual name="">
+			<visual name="base_plate_visual">
 				<origin xyz="0.0 0.0 0.0" rpy="0.0 0.0 0.0"/>
 				<geometry>
@@ -15,7 +15,7 @@
 			</visual>
 			<collision name="base_plate_collision">
-				<origin xyz="0.0 0.0 0.0" rpy="0.0 0.0 0.0"/>
+				<origin xyz="0.0 0.0125 0.0" rpy="0.0 0.0 0.0"/>
 				<geometry>
-					<box size="0.1 0.1 0.1"/>
+					<box size="0.300 0.025 0.300"/>
 				</geometry>
 			</collision>
@@ -43,10 +43,10 @@
 				<origin xyz="0.0 0.0 0.0" rpy="0.0 0.0 0.0"/>
 				<geometry>
-					<box size="0.1 0.1 0.1"/>
+						<mesh filename="package://wheel_bot_description/meshes/WheelHub.dae" />
 				</geometry>
 			</collision>
 		</link>
 		<joint name="l_hub_to_base_plate" type="fixed">
-			<origin xyz="0.1 0.025 0.150" rpy="0.0 3.14 0.0"/>
+			<origin xyz="0.050 0.025 0.140" rpy="0.0 0.0 0.0"/>
 			<parent link="base_plate_link"/>
 			<child link="l_wheel_hub"/>
@@ -67,12 +67,12 @@
 			</visual>
 			<collision name="l_wheel_bearing_collision">
-				<origin xyz="0.0 0.0 0.0" rpy="0.0 0.0 0.0"/>
+				<origin xyz="0.0 0.0 0.0" rpy="0.0 1.57075 0.0"/>
 				<geometry>
-					<box size="0.1 0.1 0.1"/>
+				<cylinder radius=".018" length="0.007"/>
 				</geometry>
 			</collision>
 		</link>
 		<joint name="l_bearing_to_hub" type="fixed">
-			<origin xyz="0.025 0.080 0.010" rpy="0.0 1.57075 0.0"/>
+			<origin xyz="0.025 0.077 0.0103" rpy="0.0 1.57075 0.0"/>
 			<parent link="l_wheel_hub"/>
 			<child link="l_wheel_bearing"/>
@@ -93,12 +93,12 @@
 			</visual>
 			<collision name="l_wheel_shaft_collision">
-				<origin xyz="0.0 0.0 0.0" rpy="0.0 0.0 0.0"/>
+				<origin xyz="0.069 0.0 0.0" rpy="0.0 -1.57075 0.0"/>
 				<geometry>
-					<box size="0.1 0.1 0.1"/>
+				<cylinder radius="0.012" length="0.100"/>
 				</geometry>
 			</collision>
 		</link>
 		<joint name="l_shaft_to_bearing" type="continuous">
-			<origin xyz="0.0 0.0 0.0" rpy="0.0 0.0 0.0"/>
+			<origin xyz="0.069 0.0 0.00" rpy="0.0 3.14159 0.0"/>
 			<parent link="l_wheel_bearing"/>
 			<child link="l_wheel_shaft"/>
@@ -129,5 +129,5 @@
 		</link>
 		<joint name="l_wheel_to_shaft" type="fixed">
-			<origin xyz="0.0 0.0 0.0" rpy="0.0 1.57075 0.0"/>
+			<origin xyz="0.100 0.0 0.0" rpy="0.0 4.712385 0.0"/>
 			<parent link="l_wheel_shaft"/>
 			<child link="l_wheel"/>

Commit message: left side completed. Both left and right side need inertias

File: catkin_ws/src/wheel_bot_description/urdf/frame.xacro (robot description, xacro)
@@ -123,7 +123,4 @@
 					<mesh filename="package://wheel_bot_description/meshes/Wheel.dae" />
 				</geometry>
-				<!-- <geometry>
-					<box size="0.1 0.1 0.1"/>
-				</geometry> -->
 			</collision>
 		</link>
@@ -135,3 +132,107 @@
 			<limit lower="0.0" upper="0.0" effort="0.0" velocity="0.0"/>
 		</joint>
+		<link name="r_wheel_hub">
+			<inertial>
+				<origin xyz="0.0 0.0 0.0" rpy="0.0 0.0 0.0"/>
+				<mass value="0.1"/>
+				<inertia ixx="0.1" ixy="0.0" ixz="0.0" iyy="0.1" iyz="0.0" izz="0.1"/>
+			</inertial>
+			<visual name="r_wheel_hub_visual">
+				<origin xyz="0.0 0.0 0.0" rpy="0.0 0.0 0.0"/>
+					<geometry>
+						<mesh filename="package://wheel_bot_description/meshes/WheelHub.dae" />
+					</geometry>
+			</visual>
+			<collision name="r_wheel_hub_collision">
+				<origin xyz="0.0 0.0 0.0" rpy="0.0 0.0 0.0"/>
+				<geometry>
+						<mesh filename="package://wheel_bot_description/meshes/WheelHub.dae" />
+				</geometry>
+			</collision>
+		</link>
+		<joint name="r_hub_to_base_plate" type="fixed">
+			<origin xyz="0.100 0.025 -0.140" rpy="0.0 3.14159 0.0"/>
+			<parent link="base_plate_link"/>
+			<child link="r_wheel_hub"/>
+			<axis xyz="0.0 0.0 0.0"/>
+			<limit lower="0.0" upper="0.0" effort="0.0" velocity="0.0"/>
+		</joint>
+		<link name="r_wheel_bearing">
+			<inertial>
+				<origin xyz="0.0 0.0 0.0" rpy="0.0 0.0 0.0"/>
+				<mass value="0.1"/>
+				<inertia ixx="0.1" ixy="0.0" ixz="0.0" iyy="0.1" iyz="0.0" izz="0.1"/>
+			</inertial>
+			<visual name="r_wheel_bearing_visual">
+				<origin xyz="0.0 0.0 0.0" rpy="0.0 0.0 0.0"/>
+					<geometry>
+						<mesh filename="package://wheel_bot_description/meshes/WheelBearing.dae" />
+					</geometry>
+			</visual>
+			<collision name="r_wheel_bearing_collision">
+				<origin xyz="0.0 0.0 0.0" rpy="0.0 1.57075 0.0"/>
+				<geometry>
+				<cylinder radius=".018" length="0.007"/>
+				</geometry>
+			</collision>
+		</link>
+		<joint name="r_bearing_to_hub" type="fixed">
+			<origin xyz="0.025 0.077 0.0103" rpy="0.0 1.57075 0.0"/>
+			<parent link="r_wheel_hub"/>
+			<child link="r_wheel_bearing"/>
+			<axis xyz="0.0 0.0 0.0"/>
+			<limit lower="0.0" upper="0.0" effort="0.0" velocity="0.0"/>
+		</joint>
+		<link name="r_wheel_shaft">
+			<inertial>
+				<origin xyz="0.0 0.0 0.0" rpy="0.0 0.0 0.0"/>
+				<mass value="0.1"/>
+				<inertia ixx="0.1" ixy="0.0" ixz="0.0" iyy="0.1" iyz="0.0" izz="0.1"/>
+			</inertial>
+			<visual name="r_wheel_shaft_visual">
+				<origin xyz="0.0 0.0 0.0" rpy="0.0 0.0 0.0"/>
+					<geometry>
+						<mesh filename="package://wheel_bot_description/meshes/WheelShaft.dae" />
+					</geometry>
+			</visual>
+			<collision name="r_wheel_shaft_collision">
+				<origin xyz="0.069 0.0 0.0" rpy="0.0 -1.57075 0.0"/>
+				<geometry>
+				<cylinder radius="0.012" length="0.100"/>
+				</geometry>
+			</collision>
+		</link>
+		<joint name="r_shaft_to_bearing" type="continuous">
+			<origin xyz="0.069 0.0 0.00" rpy="0.0 3.14159 0.0"/>
+			<parent link="r_wheel_bearing"/>
+			<child link="r_wheel_shaft"/>
+			<axis xyz="1.0 0.0 0.0"/>
+			<limit lower="0.0" upper="0.0" effort="0.0" velocity="0.0"/>
+		</joint>
+		<link name="r_wheel">
+			<inertial>
+				<origin xyz="0.0 0.0 0.0" rpy="0.0 0.0 0.0"/>
+				<mass value="0.1"/>
+				<inertia ixx="0.1" ixy="0.0" ixz="0.0" iyy="0.1" iyz="0.0" izz="0.1"/>
+			</inertial>
+			<visual name="r_wheel_visual">
+				<origin xyz="0.0 0.0 0.0" rpy="0.0 0.0 0.0"/>
+					<geometry>
+						<mesh filename="package://wheel_bot_description/meshes/Wheel.dae" />
+					</geometry>
+			</visual>
+			<collision name="r_wheel_collision">
+				<origin xyz="0.0 0.0 0.0" rpy="0.0 0.0 0.0"/>
+				<geometry>
+					<mesh filename="package://wheel_bot_description/meshes/Wheel.dae" />
+				</geometry>
+			</collision>
+		</link>
+		<joint name="r_wheel_to_shaft" type="fixed">
+			<origin xyz="0.100 0.0 0.0" rpy="0.0 4.712385 0.0"/>
+			<parent link="r_wheel_shaft"/>
+			<child link="r_wheel"/>
+			<axis xyz="0.0 0.0 0.0"/>
+			<limit lower="0.0" upper="0.0" effort="0.0" velocity="0.0"/>
+		</joint>
 </robot>

Commit message: EOD

File: catkin_ws/src/wheel_bot_description/urdf/frame.xacro (robot description, xacro)
@@ -29,4 +29,108 @@
 			<limit lower="0.0" upper="0.0" effort="0.0" velocity="0.0"/>
 		</joint>
+		<link name="r_wheel_hub">
+			<inertial>
+				<origin xyz="0.0 0.0 0.0" rpy="0.0 0.0 0.0"/>
+				<mass value="0.1"/>
+				<inertia ixx="0.1" ixy="0.0" ixz="0.0" iyy="0.1" iyz="0.0" izz="0.1"/>
+			</inertial>
+			<visual name="r_wheel_hub_visual">
+				<origin xyz="0.0 0.0 0.0" rpy="0.0 0.0 0.0"/>
+					<geometry>
+						<mesh filename="package://wheel_bot_description/meshes/WheelHub.dae" />
+					</geometry>
+			</visual>
+			<collision name="r_wheel_hub_collision">
+				<origin xyz="0.0 0.0 0.0" rpy="0.0 0.0 0.0"/>
+				<geometry>
+						<mesh filename="package://wheel_bot_description/meshes/WheelHub.dae" />
+				</geometry>
+			</collision>
+		</link>
+		<joint name="r_hub_to_base_plate" type="fixed">
+			<origin xyz="0.050 0.025 0.140" rpy="0.0 0.0 0.0"/>
+			<parent link="base_plate_link"/>
+			<child link="r_wheel_hub"/>
+			<axis xyz="0.0 0.0 0.0"/>
+			<limit lower="0.0" upper="0.0" effort="0.0" velocity="0.0"/>
+		</joint>
+		<link name="r_wheel_bearing">
+			<inertial>
+				<origin xyz="0.0 0.0 0.0" rpy="0.0 0.0 0.0"/>
+				<mass value="0.1"/>
+				<inertia ixx="0.1" ixy="0.0" ixz="0.0" iyy="0.1" iyz="0.0" izz="0.1"/>
+			</inertial>
+			<visual name="r_wheel_bearing_visual">
+				<origin xyz="0.0 0.0 0.0" rpy="0.0 0.0 0.0"/>
+					<geometry>
+						<mesh filename="package://wheel_bot_description/meshes/WheelBearing.dae" />
+					</geometry>
+			</visual>
+			<collision name="r_wheel_bearing_collision">
+				<origin xyz="0.0 0.0 0.0" rpy="0.0 1.57075 0.0"/>
+				<geometry>
+				<cylinder radius=".018" length="0.007"/>
+				</geometry>
+			</collision>
+		</link>
+		<joint name="r_bearing_to_hub" type="fixed">
+			<origin xyz="0.025 0.077 0.0103" rpy="0.0 1.57075 0.0"/>
+			<parent link="r_wheel_hub"/>
+			<child link="r_wheel_bearing"/>
+			<axis xyz="0.0 0.0 0.0"/>
+			<limit lower="0.0" upper="0.0" effort="0.0" velocity="0.0"/>
+		</joint>
+		<link name="r_wheel_shaft">
+			<inertial>
+				<origin xyz="0.0 0.0 0.0" rpy="0.0 0.0 0.0"/>
+				<mass value="0.1"/>
+				<inertia ixx="0.1" ixy="0.0" ixz="0.0" iyy="0.1" iyz="0.0" izz="0.1"/>
+			</inertial>
+			<visual name="r_wheel_shaft_visual">
+				<origin xyz="0.0 0.0 0.0" rpy="0.0 0.0 0.0"/>
+					<geometry>
+						<mesh filename="package://wheel_bot_description/meshes/WheelShaft.dae" />
+					</geometry>
+			</visual>
+			<collision name="r_wheel_shaft_collision">
+				<origin xyz="0.069 0.0 0.0" rpy="0.0 -1.57075 0.0"/>
+				<geometry>
+				<cylinder radius="0.012" length="0.100"/>
+				</geometry>
+			</collision>
+		</link>
+		<joint name="r_shaft_to_bearing" type="continuous">
+			<origin xyz="0.069 0.0 0.00" rpy="0.0 3.14159 0.0"/>
+			<parent link="r_wheel_bearing"/>
+			<child link="r_wheel_shaft"/>
+			<axis xyz="1.0 0.0 0.0"/>
+			<limit lower="0.0" upper="0.0" effort="0.0" velocity="0.0"/>
+		</joint>
+		<link name="r_wheel">
+			<inertial>
+				<origin xyz="0.0 0.0 0.0" rpy="0.0 0.0 0.0"/>
+				<mass value="0.1"/>
+				<inertia ixx="0.1" ixy="0.0" ixz="0.0" iyy="0.1" iyz="0.0" izz="0.1"/>
+			</inertial>
+			<visual name="r_wheel_visual">
+				<origin xyz="0.0 0.0 0.0" rpy="0.0 0.0 0.0"/>
+					<geometry>
+						<mesh filename="package://wheel_bot_description/meshes/Wheel.dae" />
+					</geometry>
+			</visual>
+			<collision name="r_wheel_collision">
+				<origin xyz="0.0 0.0 0.0" rpy="0.0 0.0 0.0"/>
+				<geometry>
+					<mesh filename="package://wheel_bot_description/meshes/Wheel.dae" />
+				</geometry>
+			</collision>
+		</link>
+		<joint name="r_wheel_to_shaft" type="fixed">
+			<origin xyz="0.100 0.0 0.0" rpy="0.0 4.712385 0.0"/>
+			<parent link="r_wheel_shaft"/>
+			<child link="r_wheel"/>
+			<axis xyz="0.0 0.0 0.0"/>
+			<limit lower="0.0" upper="0.0" effort="0.0" velocity="0.0"/>
+		</joint>
 		<link name="l_wheel_hub">
 			<inertial>
@@ -49,5 +153,5 @@
 		</link>
 		<joint name="l_hub_to_base_plate" type="fixed">
-			<origin xyz="0.050 0.025 0.140" rpy="0.0 0.0 0.0"/>
+			<origin xyz="0.100 0.025 -0.140" rpy="0.0 3.14159 0.0"/>
 			<parent link="base_plate_link"/>
 			<child link="l_wheel_hub"/>
@@ -133,105 +237,57 @@
 			<limit lower="0.0" upper="0.0" effort="0.0" velocity="0.0"/>
 		</joint>
-		<link name="r_wheel_hub">
-			<inertial>
-				<origin xyz="0.0 0.0 0.0" rpy="0.0 0.0 0.0"/>
-				<mass value="0.1"/>
-				<inertia ixx="0.1" ixy="0.0" ixz="0.0" iyy="0.1" iyz="0.0" izz="0.1"/>
-			</inertial>
-			<visual name="r_wheel_hub_visual">
-				<origin xyz="0.0 0.0 0.0" rpy="0.0 0.0 0.0"/>
-					<geometry>
-						<mesh filename="package://wheel_bot_description/meshes/WheelHub.dae" />
-					</geometry>
-			</visual>
-			<collision name="r_wheel_hub_collision">
-				<origin xyz="0.0 0.0 0.0" rpy="0.0 0.0 0.0"/>
-				<geometry>
-						<mesh filename="package://wheel_bot_description/meshes/WheelHub.dae" />
-				</geometry>
-			</collision>
-		</link>
-		<joint name="r_hub_to_base_plate" type="fixed">
-			<origin xyz="0.100 0.025 -0.140" rpy="0.0 3.14159 0.0"/>
+		<link name="camera">
+			<inertial>
+				<origin xyz="0.0 0.0 0.0" rpy="0.0 0.0 0.0"/>
+				<mass value="0.1"/>
+				<inertia ixx="1e-6" ixy="0.0" ixz="0.0" iyy="1e-6" iyz="0.0" izz="1e-6"/>
+			</inertial>
+			<visual name="camera_visual">
+				<origin xyz="0.0 0.0 0.0" rpy="0.0 0.0 0.0"/>
+				<geometry>
+					<box size="0.05 0.05 0.05"/>
+				</geometry>
+				<material name="">
+					<color rgba="1.0 0.0 0.0 1.0"/>
+					<texture filename=""/>
+				</material>
+			</visual>
+			<collision name="camera_collision">
+				<origin xyz="0.0 0.0 0.0" rpy="0.0 0.0 0.0"/>
+				<geometry>
+					<box size="0.05 0.05 0.05"/>
+				</geometry>
+			</collision>
+		</link>
+		<joint name="camera_to_base" type="fixed">
+			<origin xyz="0.1 0.050 0.0" rpy="-1.57075 0.0 0.0"/>
 			<parent link="base_plate_link"/>
-			<child link="r_wheel_hub"/>
-			<axis xyz="0.0 0.0 0.0"/>
-			<limit lower="0.0" upper="0.0" effort="0.0" velocity="0.0"/>
-		</joint>
-		<link name="r_wheel_bearing">
-			<inertial>
-				<origin xyz="0.0 0.0 0.0" rpy="0.0 0.0 0.0"/>
-				<mass value="0.1"/>
-				<inertia ixx="0.1" ixy="0.0" ixz="0.0" iyy="0.1" iyz="0.0" izz="0.1"/>
-			</inertial>
-			<visual name="r_wheel_bearing_visual">
-				<origin xyz="0.0 0.0 0.0" rpy="0.0 0.0 0.0"/>
-					<geometry>
-						<mesh filename="package://wheel_bot_description/meshes/WheelBearing.dae" />
-					</geometry>
-			</visual>
-			<collision name="r_wheel_bearing_collision">
-				<origin xyz="0.0 0.0 0.0" rpy="0.0 1.57075 0.0"/>
-				<geometry>
-				<cylinder radius=".018" length="0.007"/>
-				</geometry>
-			</collision>
-		</link>
-		<joint name="r_bearing_to_hub" type="fixed">
-			<origin xyz="0.025 0.077 0.0103" rpy="0.0 1.57075 0.0"/>
-			<parent link="r_wheel_hub"/>
-			<child link="r_wheel_bearing"/>
-			<axis xyz="0.0 0.0 0.0"/>
-			<limit lower="0.0" upper="0.0" effort="0.0" velocity="0.0"/>
-		</joint>
-		<link name="r_wheel_shaft">
-			<inertial>
-				<origin xyz="0.0 0.0 0.0" rpy="0.0 0.0 0.0"/>
-				<mass value="0.1"/>
-				<inertia ixx="0.1" ixy="0.0" ixz="0.0" iyy="0.1" iyz="0.0" izz="0.1"/>
-			</inertial>
-			<visual name="r_wheel_shaft_visual">
-				<origin xyz="0.0 0.0 0.0" rpy="0.0 0.0 0.0"/>
-					<geometry>
-						<mesh filename="package://wheel_bot_description/meshes/WheelShaft.dae" />
-					</geometry>
-			</visual>
-			<collision name="r_wheel_shaft_collision">
-				<origin xyz="0.069 0.0 0.0" rpy="0.0 -1.57075 0.0"/>
-				<geometry>
-				<cylinder radius="0.012" length="0.100"/>
-				</geometry>
-			</collision>
-		</link>
-		<joint name="r_shaft_to_bearing" type="continuous">
-			<origin xyz="0.069 0.0 0.00" rpy="0.0 3.14159 0.0"/>
-			<parent link="r_wheel_bearing"/>
-			<child link="r_wheel_shaft"/>
-			<axis xyz="1.0 0.0 0.0"/>
-			<limit lower="0.0" upper="0.0" effort="0.0" velocity="0.0"/>
-		</joint>
-		<link name="r_wheel">
-			<inertial>
-				<origin xyz="0.0 0.0 0.0" rpy="0.0 0.0 0.0"/>
-				<mass value="0.1"/>
-				<inertia ixx="0.1" ixy="0.0" ixz="0.0" iyy="0.1" iyz="0.0" izz="0.1"/>
-			</inertial>
-			<visual name="r_wheel_visual">
-				<origin xyz="0.0 0.0 0.0" rpy="0.0 0.0 0.0"/>
-					<geometry>
-						<mesh filename="package://wheel_bot_description/meshes/Wheel.dae" />
-					</geometry>
-			</visual>
-			<collision name="r_wheel_collision">
-				<origin xyz="0.0 0.0 0.0" rpy="0.0 0.0 0.0"/>
-				<geometry>
-					<mesh filename="package://wheel_bot_description/meshes/Wheel.dae" />
-				</geometry>
-			</collision>
-		</link>
-		<joint name="r_wheel_to_shaft" type="fixed">
-			<origin xyz="0.100 0.0 0.0" rpy="0.0 4.712385 0.0"/>
-			<parent link="r_wheel_shaft"/>
-			<child link="r_wheel"/>
+			<child link="camera"/>
+			<axis xyz="0.0 0.0 0.0"/>
+			<limit lower="0.0" upper="0.0" effort="0.0" velocity="0.0"/>
+		</joint>
+		<link name="hokuyo">
+			<inertial>
+				<origin xyz="0.0 0.0 0.0" rpy="0.0 0.0 0.0"/>
+				<mass value="0.1"/>
+				<inertia ixx="1e-6" ixy="0.0" ixz="0.0" iyy="1e-6" iyz="0.0" izz="1e-6"/>
+			</inertial>
+			<visual name="hokuyo_visual">
+				<origin xyz="0.0 0.0 0.0" rpy="0.0 0.0 0.0"/>
+				<geometry>
+					<mesh filename="package://wheel_bot_description/meshes/hokuyo.dae"/>
+				</geometry>
+			</visual>
+			<collision>
+				<origin xyz="0.0 0.0 0.0" rpy="0.0 0.0 0.0"/>
+				<geometry>
+					<box size="0.05 0.05 0.05"/>
+				</geometry>
+			</collision>
+		</link>
+		<joint name="hokuyo_to_camera" type="fixed">
+			<origin xyz="0.0 0.0 0.060" rpy="0.0 0.0 0.0"/>
+			<parent link="camera"/>
+			<child link="hokuyo"/>
 			<axis xyz="0.0 0.0 0.0"/>
 			<limit lower="0.0" upper="0.0" effort="0.0" velocity="0.0"/>
